File: KiCAD/LDC_TIA/LDC_TIA.kicad_pcb_v1.kicad_pcb (KiCad board)
At the start: 2 copper layers, 57 x 29.6 mm, 23 parts, among them J1 54-00166, J2 Conn_01x07_Pin, J3 Conn_01x02_Pin, Q1 BC817, SW2 B3F-6020, U1 OPA2197xD, U2 LTC1044, U3 LM7805_TO220

Commit message: pcb v4
Routing:
- net /-VCC: track 59.0 -> 58.2 mm
Other:
- board size 57 x 29.6 mm -> 57 x 32.8 mm
Changed lines of the file:
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@@
 		)
 	)
-	(gr_rect
-		(start 78.705 58.08)
-		(end 135.72 87.64)
+	(gr_circle
+		(center 133.47 88.75)
+		(end 134.97 88.75)
 		(stroke
 			(width 0.05)
@@
 		(layer "Edge.Cuts")
 	)
+	(gr_circle
+		(center 133.58 60.02)
+		(end 135.08 60.02)
+		(stroke
+			(width 0.05)
+			(type solid)
+		)
+		(fill no)
+		(layer "Edge.Cuts")
+	)
+	(gr_circle
+		(center 80.88 60.36)
+		(end 82.38 60.36)
+		(stroke
+			(width 0.05)
+			(type solid)
+		)
+		(fill no)
+		(layer "Edge.Cuts")
+	)
+	(gr_circle
+		(center 80.74 88.77)
+		(end 82.24 88.77)
+		(stroke
+			(width 0.05)
+			(type solid)
+		)
+		(fill no)
+		(layer "Edge.Cuts")
+	)
+	(gr_rect
+		(start 78.705 58.08)
+		(end 135.72 90.91)
+		(stroke
+			(width 0.05)
+			(type solid)
+		)
+		(fill no)
+		(layer "Edge.Cuts")
+	)
 	(gr_text "LDC+TIA: Version V1\nMegha, Project Associate, IITM"
 		(at 80.3925 86.66 0)
@@
 	)
 	(gr_text "CATHOD"
-		(at 128.85 84.87 0)
+		(at 128.75 85.27 0)
 		(layer "F.SilkS")
 		(effects
@@
 	)
 	(segment
+		(start 129.61 86.77)
+		(end 134.96 81.42)
+		(width 0.2)
+		(layer "F.Cu")
+		(net 9)
+	)
+	(segment
+		(start 120.911 86.77)
+		(end 129.61 86.77)
+		(width 0.2)
+		(layer "F.Cu")
+		(net 9)
+	)
+	(segment
+		(start 117.931899 77.514)
+		(end 118.749 78.331101)
+		(width 0.2)
+		(layer "F.Cu")
+		(net 9)
+	)
+	(segment
+		(start 111.82 78.2)
+		(end 111.905 78.115)
+		(width 0.2)
+		(layer "F.Cu")
+		(net 9)
+	)
+	(segment
+		(start 111.82 80.16)
+		(end 111.82 78.2)
+		(width 0.2)
+		(layer "F.Cu")
+		(net 9)
+	)
+	(segment
+		(start 118.749 84.608)
+		(end 120.911 86.77)
+		(width 0.2)
+		(layer "F.Cu")
+		(net 9)
+	)
+	(segment
+		(start 112.506 77.514)
+		(end 117.931899 77.514)
+		(width 0.2)
+		(layer "F.Cu")
+		(net 9)
+	)
+	(segment
+		(start 103.38 82.35)
+		(end 105.57 80.16)
+		(width 0.2)
+		(layer "F.Cu")
+		(net 9)
+	)
+	(segment
+		(start 134.96 81.42)
+		(end 134.96 76.46)
+		(width 0.2)
+		(layer "F.Cu")
+		(net 9)
+	)
+	(segment
+		(start 133.13 74.63)
+		(end 126.95 74.63)
+		(width 0.2)
+		(layer "F.Cu")
+		(net 9)
+	)
+	(segment
 		(start 111.905 78.115)
 		(end 112.506 77.514)
@@
 	)
 	(segment
-		(start 112.506 77.514)
-		(end 117.931899 77.514)
-		(width 0.2)
-		(layer "F.Cu")
-		(net 9)
-	)
-	(segment
-		(start 111.82 78.2)
-		(end 111.905 78.115)
-		(width 0.2)
-		(layer "F.Cu")
-		(net 9)
-	)
-	(segment
-		(start 111.82 80.16)
-		(end 111.82 78.2)
+		(start 105.57 80.16)
+		(end 111.82 80.16)
 		(width 0.2)
 		(layer "F.Cu")
@@
 		(width 0.2)
 		(layer "F.Cu")
-		(net 9)
-	)
-	(segment
-		(start 118.749 84.608)
-		(end 120.911 86.77)
-		(width 0.2)
-		(layer "F.Cu")
-		(net 9)
-	)
-	(segment
-		(start 117.931899 77.514)
-		(end 118.749 78.331101)
-		(width 0.2)
-		(layer "F.Cu")
-		(net 9)
-	)
-	(segment
-		(start 103.38 82.35)
-		(end 105.57 80.16)
-		(width 0.2)
-		(layer "F.Cu")
-		(net 9)
-	)
-	(segment
-		(start 120.911 86.77)
-		(end 131.03 86.77)
-		(width 0.2)
-		(layer "F.Cu")
-		(net 9)
-	)
-	(segment
-		(start 134.96 82.84)
-		(end 134.96 76.46)
-		(width 0.2)
-		(layer "F.Cu")
-		(net 9)
-	)
-	(segment
-		(start 133.13 74.63)
-		(end 126.95 74.63)
-		(width 0.2)
-		(layer "F.Cu")
-		(net 9)
-	)
-	(segment
-		(start 131.03 86.77)
-		(end 134.96 82.84)
-		(width 0.2)
-		(layer "F.Cu")
-		(net 9)
-	)
-	(segment
-		(start 105.57 80.16)
-		(end 111.82 80.16)
-		(width 0.2)
-		(layer "F.Cu")
